File: empty_shield/Empty_Shield_SMD-v13.brd (EAGLE design)
At the start: 101.6 x 53.3 mm, 18 parts

Commit message: empty shield SMD
Parts:
- LED1, LED2: device SparkFun:LED5MM -> led:CHIP-LED0805
- R1, R2, R3: device SparkFun:AXIAL-0.3 -> rcl:R0805
Connections:
- net 5V: now also R1.2, R3.2; no longer R1.P$2, R3.P$2
- net D13: now also R2.2; no longer R2.P$2
- net GND: now also LED1.C, LED2.C; no longer LED1.K, LED2.K
- net N$126: now also R1.1; no longer R1.P$1
- net N$127: now also R2.1; no longer R2.P$1
- net RES: now also R3.1; no longer R3.P$1
Changed lines of the file:
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@@
 <element name="JP12" library="SparkFun" package="1X02_LOCK" value="" x="93.98" y="50.8"/>
 <element name="S1" library="SparkFun" package="TACTILE-PTH" value="" x="27.94" y="4.826" rot="R270"/>
-<element name="LED1" library="SparkFun" package="LED5MM" value="Red" x="10.16" y="5.08" rot="R180"/>
-<element name="LED2" library="SparkFun" package="LED5MM" value="Green" x="3.81" y="5.08"/>
-<element name="R1" library="SparkFun" package="AXIAL-0.3" value="330" x="19.05" y="7.747"/>
-<element name="R2" library="SparkFun" package="AXIAL-0.3" value="330" x="19.05" y="10.16"/>
-<element name="R3" library="SparkFun" package="AXIAL-0.3" value="10k" x="19.05" y="5.461" smashed="yes" rot="R180">
+<element name="LED1" library="led" package="CHIP-LED0805" value="Red" x="10.16" y="5.08" rot="R180"/>
+<element name="LED2" library="led" package="CHIP-LED0805" value="Green" x="3.81" y="5.08"/>
+<element name="R1" library="rcl" package="R0805" value="330" x="19.05" y="7.747"/>
+<element name="R2" library="rcl" package="R0805" value="330" x="19.05" y="10.16"/>
+<element name="R3" library="rcl" package="R0805" value="10k" x="19.05" y="5.461" smashed="yes" rot="R180">
 <attribute name="NAME" x="21.59" y="4.191" size="0.4064" layer="25" rot="R180"/>
 <attribute name="VALUE" x="19.177" y="5.969" size="0.8128" layer="21" ratio="15" rot="R180"/>
@@
 <signal name="RES">
 <contactref element="JP10" pad="1"/>
-<contactref element="R3" pad="P$1"/>
+<contactref element="R3" pad="1"/>
 <contactref element="S1" pad="4"/>
 <contactref element="S1" pad="3"/>
 <wire x1="25.6794" y1="1.5748" x2="33.02" y2="2.54" width="0" layer="19" extent="1-1"/>
-<wire x1="22.86" y1="5.461" x2="25.6794" y2="1.5748" width="0" layer="19" extent="1-1"/>
-<wire x1="25.6794" y1="8.0772" x2="22.86" y2="5.461" width="0" layer="19" extent="1-1"/>
+<wire x1="20" y1="5.461" x2="25.6794" y2="1.5748" width="0" layer="19" extent="1-1"/>
+<wire x1="25.6794" y1="8.0772" x2="20" y2="5.461" width="0" layer="19" extent="1-1"/>
 </signal>
 <signal name="3.3">
@@
 <signal name="5V">
 <contactref element="JP10" pad="3"/>
-<contactref element="R3" pad="P$2"/>
-<contactref element="R1" pad="P$2"/>
-<wire x1="22.86" y1="7.747" x2="38.1" y2="2.54" width="0" layer="19" extent="1-1"/>
-<wire x1="15.24" y1="5.461" x2="22.86" y2="7.747" width="0" layer="19" extent="1-1"/>
+<contactref element="R3" pad="2"/>
+<contactref element="R1" pad="2"/>
+<wire x1="20" y1="7.747" x2="38.1" y2="2.54" width="0" layer="19" extent="1-1"/>
+<wire x1="18.1" y1="5.461" x2="20" y2="7.747" width="0" layer="19" extent="1-1"/>
 </signal>
 <signal name="GND">
@@
 <contactref element="S1" pad="1"/>
 <contactref element="S1" pad="2"/>
-<contactref element="LED1" pad="K"/>
-<contactref element="LED2" pad="K"/>
+<contactref element="LED1" pad="C"/>
+<contactref element="LED2" pad="C"/>
 <contactref element="JP3" pad="7"/>
 <contactref element="JP11" pad="1"/>
@@
 <wire x1="30.2006" y1="1.5748" x2="40.64" y2="2.286" width="0" layer="19" extent="1-1"/>
 <wire x1="30.2006" y1="8.0772" x2="30.2006" y2="1.5748" width="0" layer="19" extent="1-1"/>
-<wire x1="8.89" y1="5.08" x2="30.2006" y2="8.0772" width="0" layer="19" extent="1-1"/>
-<wire x1="5.08" y1="5.08" x2="8.89" y2="5.08" width="0" layer="19" extent="1-1"/>
+<wire x1="10.16" y1="4.03" x2="30.2006" y2="8.0772" width="0" layer="19" extent="1-1"/>
+<wire x1="3.81" y1="6.13" x2="10.16" y2="4.03" width="0" layer="19" extent="1-1"/>
 <wire x1="26.67" y1="50.673" x2="30.2006" y2="8.0772" width="0" layer="19" extent="1-1"/>
 </signal>
@@
 <signal name="D13">
 <contactref element="JP3" pad="6"/>
-<contactref element="R2" pad="P$2"/>
-<wire x1="22.86" y1="10.16" x2="29.21" y2="50.927" width="0" layer="19" extent="1-1"/>
+<contactref element="R2" pad="2"/>
+<wire x1="20" y1="10.16" x2="29.21" y2="50.927" width="0" layer="19" extent="1-1"/>
 </signal>
 <signal name="AREF">
@@
 </signal>
 <signal name="N$126">
-<contactref element="R1" pad="P$1"/>
+<contactref element="R1" pad="1"/>
 <contactref element="LED1" pad="A"/>
-<wire x1="11.43" y1="5.08" x2="15.24" y2="7.747" width="0" layer="19" extent="1-1"/>
+<wire x1="10.16" y1="6.13" x2="18.1" y2="7.747" width="0" layer="19" extent="1-1"/>
 </signal>
 <signal name="N$127">
-<contactref element="R2" pad="P$1"/>
+<contactref element="R2" pad="1"/>
 <contactref element="LED2" pad="A"/>
-<wire x1="2.54" y1="5.08" x2="15.24" y2="10.16" width="0" layer="19" extent="1-1"/>
-</signal>
-<signal name="N$319">
-<via x="38.1" y="7.62" extent="1-16" drill="1.016" diameter="1.8796"/>
-</signal>
-<signal name="N$320">
-<via x="40.64" y="7.62" extent="1-16" drill="1.016" diameter="1.8796"/>
-</signal>
-<signal name="N$321">
-<via x="43.18" y="7.62" extent="1-16" drill="1.016" diameter="1.8796"/>
-</signal>
-<signal name="N$322">
-<via x="48.26" y="7.62" extent="1-16" drill="1.016" diameter="1.8796"/>
-</signal>
-<signal name="N$323">
-<via x="45.72" y="7.62" extent="1-16" drill="1.016" diameter="1.8796"/>
+<wire x1="3.81" y1="4.03" x2="18.1" y2="10.16" width="0" layer="19" extent="1-1"/>
 </signal>
 </signals>

Commit message: Empty MEGA SMD shield template
Parts:
- moved R2 11.5 mm to (7.62, 8.89)
- moved R1 5.24 mm to (14.0, 9.02)
- moved R3 5.24 mm to (14.0, 6.73)
- moved S1 1.27 mm to (27.9, 6.10)
- turned LED2 to 180 degrees
Routing:
- net D13: track 0.00 -> 50.6 mm
- net 5V: track 0.00 -> 33.3 mm
- net RES: track 0.00 -> 25.8 mm
- net N$126: track 0.00 -> 4.07 mm
- net N$127: track 0.00 -> 3.98 mm
- net 5V@1: track 0.00 -> 3.12 mm
Changed lines of the file:
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@@
 <setting verticaltext="up"/>
 </settings>
-<grid distance="0.05" unitdist="inch" unit="inch" style="lines" multiple="1" display="yes" altdistance="0.005" altunitdist="inch" altunit="inch"/>
+<grid distance="0.05" unitdist="inch" unit="mm" style="lines" multiple="1" display="yes" altdistance="0.005" altunitdist="inch" altunit="mm"/>
 <layers>
 <layer number="1" name="Top" color="4" fill="1" visible="yes" active="yes"/>
@@
 <element name="JP11" library="SparkFun" package="1X02_LOCK" value="" x="93.98" y="7.62"/>
 <element name="JP12" library="SparkFun" package="1X02_LOCK" value="" x="93.98" y="50.8"/>
-<element name="S1" library="SparkFun" package="TACTILE-PTH" value="" x="27.94" y="4.826" rot="R270"/>
+<element name="S1" library="SparkFun" package="TACTILE-PTH" value="" x="27.94" y="6.096" rot="R270"/>
 <element name="LED1" library="led" package="CHIP-LED0805" value="Red" x="10.16" y="5.08" rot="R180"/>
-<element name="LED2" library="led" package="CHIP-LED0805" value="Green" x="3.81" y="5.08"/>
-<element name="R1" library="rcl" package="R0805" value="330" x="19.05" y="7.747"/>
-<element name="R2" library="rcl" package="R0805" value="330" x="19.05" y="10.16"/>
-<element name="R3" library="rcl" package="R0805" value="10k" x="19.05" y="5.461" smashed="yes" rot="R180">
-<attribute name="NAME" x="21.59" y="4.191" size="0.4064" layer="25" rot="R180"/>
-<attribute name="VALUE" x="19.177" y="5.969" size="0.8128" layer="21" ratio="15" rot="R180"/>
+<element name="LED2" library="led" package="CHIP-LED0805" value="Green" x="3.81" y="5.08" rot="R180"/>
+<element name="R1" library="rcl" package="R0805" value="330" x="13.97" y="9.017"/>
+<element name="R2" library="rcl" package="R0805" value="330" x="7.62" y="8.89"/>
+<element name="R3" library="rcl" package="R0805" value="10k" x="13.97" y="6.731" smashed="yes" rot="R180">
+<attribute name="NAME" x="16.51" y="5.461" size="0.4064" layer="25" rot="R180"/>
+<attribute name="VALUE" x="14.097" y="7.239" size="0.8128" layer="21" ratio="15" rot="R180"/>
 </element>
 <element name="U$2" library="SparkFun" package="CREATIVE_COMMONS" value="CREATIVE_COMMONS" x="20.32" y="-7.62"/>
@@
 <contactref element="S1" pad="4"/>
 <contactref element="S1" pad="3"/>
-<wire x1="25.6794" y1="1.5748" x2="33.02" y2="2.54" width="0" layer="19" extent="1-1"/>
-<wire x1="20" y1="5.461" x2="25.6794" y2="1.5748" width="0" layer="19" extent="1-1"/>
-<wire x1="25.6794" y1="8.0772" x2="20" y2="5.461" width="0" layer="19" extent="1-1"/>
+<wire x1="25.5" y1="6.75" x2="15" y2="6.75" width="0.2032" layer="1"/>
+<wire x1="25.5" y1="9.25" x2="25.5" y2="6.75" width="0.2032" layer="1"/>
+<wire x1="15" y1="6.75" x2="14.92" y2="6.731" width="0.2032" layer="1"/>
+<wire x1="25.5" y1="9.25" x2="25.6794" y2="9.3472" width="0.2032" layer="1"/>
+<wire x1="25.5" y1="6.75" x2="25.5" y2="4.75" width="0.2032" layer="1"/>
+<wire x1="25.5" y1="4.75" x2="25.5" y2="3" width="0.2032" layer="1"/>
+<wire x1="25.5" y1="3" x2="25.6794" y2="2.8448" width="0.2032" layer="1"/>
+<wire x1="31" y1="4.75" x2="33" y2="2.75" width="0.2032" layer="1"/>
+<wire x1="25.5" y1="4.75" x2="31" y2="4.75" width="0.2032" layer="1"/>
+<wire x1="33" y1="2.75" x2="33.02" y2="2.54" width="0.2032" layer="1"/>
 </signal>
 <signal name="3.3">
@@
 <contactref element="R3" pad="2"/>
 <contactref element="R1" pad="2"/>
-<wire x1="20" y1="7.747" x2="38.1" y2="2.54" width="0" layer="19" extent="1-1"/>
-<wire x1="18.1" y1="5.461" x2="20" y2="7.747" width="0" layer="19" extent="1-1"/>
+<wire x1="13.75" y1="7.25" x2="13.25" y2="6.75" width="0.2032" layer="1"/>
+<wire x1="13.75" y1="7.75" x2="13.75" y2="7.25" width="0.2032" layer="1"/>
+<wire x1="14.75" y1="8.75" x2="13.75" y2="7.75" width="0.2032" layer="1"/>
+<wire x1="14.75" y1="9" x2="14.75" y2="8.75" width="0.2032" layer="1"/>
+<wire x1="13.25" y1="6.75" x2="13.02" y2="6.731" width="0.2032" layer="1"/>
+<wire x1="14.75" y1="9" x2="14.92" y2="9.017" width="0.2032" layer="1"/>
+<wire x1="17" y1="11.25" x2="15" y2="9.25" width="0.2032" layer="1"/>
+<wire x1="28.5" y1="11.25" x2="17" y2="11.25" width="0.2032" layer="1"/>
+<wire x1="28.5" y1="8.5" x2="28.5" y2="11.25" width="0.2032" layer="1"/>
+<wire x1="32.5" y1="4.5" x2="28.5" y2="8.5" width="0.2032" layer="1"/>
+<wire x1="37.25" y1="4.5" x2="32.5" y2="4.5" width="0.2032" layer="1"/>
+<wire x1="37.25" y1="3.75" x2="37.25" y2="4.5" width="0.2032" layer="1"/>
+<wire x1="38" y1="3" x2="37.25" y2="3.75" width="0.2032" layer="1"/>
+<wire x1="38" y1="2.75" x2="38" y2="3" width="0.2032" layer="1"/>
+<wire x1="15" y1="9.25" x2="14.92" y2="9.017" width="0.2032" layer="1"/>
+<wire x1="38" y1="2.75" x2="38.1" y2="2.54" width="0.2032" layer="1"/>
 </signal>
 <signal name="GND">
@@
 <vertex x="0" y="2.54"/>
 </polygon>
-<wire x1="93.8022" y1="7.62" x2="96.6978" y2="7.62" width="0" layer="19" extent="1-1"/>
-<wire x1="43.18" y1="2.54" x2="93.8022" y2="7.62" width="0" layer="19" extent="1-1"/>
-<wire x1="40.64" y1="2.286" x2="43.18" y2="2.54" width="0" layer="19" extent="1-1"/>
-<wire x1="30.2006" y1="1.5748" x2="40.64" y2="2.286" width="0" layer="19" extent="1-1"/>
-<wire x1="30.2006" y1="8.0772" x2="30.2006" y2="1.5748" width="0" layer="19" extent="1-1"/>
-<wire x1="10.16" y1="4.03" x2="30.2006" y2="8.0772" width="0" layer="19" extent="1-1"/>
-<wire x1="3.81" y1="6.13" x2="10.16" y2="4.03" width="0" layer="19" extent="1-1"/>
-<wire x1="26.67" y1="50.673" x2="30.2006" y2="8.0772" width="0" layer="19" extent="1-1"/>
 </signal>
 <signal name="VIN">
@@
 <contactref element="JP3" pad="6"/>
 <contactref element="R2" pad="2"/>
-<wire x1="20" y1="10.16" x2="29.21" y2="50.927" width="0" layer="19" extent="1-1"/>
+<wire x1="29" y1="29.25" x2="8.75" y2="9" width="0.2032" layer="1"/>
+<wire x1="29" y1="50.75" x2="29" y2="29.25" width="0.2032" layer="1"/>
+<wire x1="8.75" y1="9" x2="8.57" y2="8.89" width="0.2032" layer="1"/>
+<wire x1="29" y1="50.75" x2="29.21" y2="50.927" width="0.2032" layer="1"/>
 </signal>
 <signal name="AREF">
@@
 <contactref element="JP12" pad="2"/>
 <contactref element="JP12" pad="1"/>
-<wire x1="93.8022" y1="50.8" x2="96.6978" y2="50.8" width="0" layer="19" extent="1-1"/>
+<wire x1="94.25" y1="50.5" x2="94" y2="50.75" width="0.2032" layer="16"/>
+<wire x1="96.25" y1="50.5" x2="94.25" y2="50.5" width="0.2032" layer="16"/>
+<wire x1="96.5" y1="50.75" x2="96.25" y2="50.5" width="0.2032" layer="16"/>
+<wire x1="94" y1="50.75" x2="93.8022" y2="50.8" width="0.2032" layer="16"/>
+<wire x1="96.5" y1="50.75" x2="96.6978" y2="50.8" width="0.2032" layer="16"/>
 </signal>
 <signal name="D22">
@@
 <contactref element="R1" pad="1"/>
 <contactref element="LED1" pad="A"/>
-<wire x1="10.16" y1="6.13" x2="18.1" y2="7.747" width="0" layer="19" extent="1-1"/>
+<wire x1="13" y1="9" x2="10.25" y2="6.25" width="0.2032" layer="1"/>
+<wire x1="10.25" y1="6.25" x2="10.16" y2="6.13" width="0.2032" layer="1"/>
+<wire x1="13" y1="9" x2="13.02" y2="9.017" width="0.2032" layer="1"/>
 </signal>
 <signal name="N$127">
 <contactref element="R2" pad="1"/>
 <contactref element="LED2" pad="A"/>
-<wire x1="3.81" y1="4.03" x2="18.1" y2="10.16" width="0" layer="19" extent="1-1"/>
+<wire x1="6.5" y1="8.75" x2="4" y2="6.25" width="0.2032" layer="1"/>
+<wire x1="4" y1="6.25" x2="3.81" y2="6.13" width="0.2032" layer="1"/>
+<wire x1="6.5" y1="8.75" x2="6.67" y2="8.89" width="0.2032" layer="1"/>
 </signal>
 </signals>
